File: board/business-card.sch (KiCad schematic (older format))
At the start: 2 parts

Commit message: schematic
Parts:
- added BT?: Battery_Cell, symbol Device:Battery_Cell
- added C? (x2): 0.1 uF, symbol Device:C
- added C?: C, symbol Device:C
- added J?: Conn_01x04, symbol Connector_Generic:Conn_01x04
- added R?: 10 K, symbol Device:R
- added SW?: SW_SPST, symbol Switch:SW_SPST
Connections:
- net SCL: now also U?.1 (SCL)
- net SDA: now also U?.4 (SDA)
- net NRESET: now reaches U?.1 (NRST)
- net NRESET: now also J?.3 (Pin_3), R?.1
- net SWIM: now reaches U?.15 (PD1)
- net SWIM: now also J?.2 (Pin_2)
- net GND: now reaches U?.4 (VSS)
- net GND: now also U?.6 (GND), U?.8 (GND), BT?.2 (-), C?.2, C?.2, C?.2, J?.4 (Pin_4)
- net at U?.5 (VCAP): now also C?.1
- net VDD: now reaches U?.6 (VDD)
- net VDD: now also U?.10 (IO_VDD), U?.9 (VDD), C?.1, C?.1, J?.1 (Pin_1), R?.2, SW?.1 (A)
- new net: BT?.1 (+), SW?.2 (B)
Changed lines of the file:
@@
 EESchema Schematic File Version 4
+LIBS:business-card-cache
 EELAYER 30 0
 EELAYER END
 $Descr A4 11693 8268
 encoding utf-8
-Sheet 1 2
+Sheet 1 1
 Title ""
 Date ""
@@
 U 1 1 5DC749E4
 P 5650 3600
-F 0 "U?" H 5650 4781 50  0000 C CNN
-F 1 "STM8S003F3U" H 5650 4690 50  0000 C CNN
+F 0 "U?" H 5300 4550 50  0000 C CNN
+F 1 "STM8S003F3U" H 5800 3150 50  0000 C CNN
 F 2 "Package_DFN_QFN:ST_UFQFPN-20_3x3mm_P0.5mm" H 5700 4700 50  0001 L CNN
 F 3 "http://www.st.com/st-web-ui/static/active/en/resource/technical/document/datasheet/DM00024550.pdf" H 5600 3200 50  0001 C CNN
@@
 	1    0    0    -1
 $EndComp
-Wire Wire Line
-	5050 3300 4950 3300
-Wire Wire Line
-	5050 3400 4950 3400
-Text HLabel 4950 3300 0    50   Input ~ 0
+Text HLabel 5000 3300 0    50   Input ~ 0
 SCL
-Text HLabel 4950 3400 0    50   Input ~ 0
+Text HLabel 5000 3400 0    50   Input ~ 0
 SDA
 $Comp
@@
 	1    0    0    -1
 $EndComp
+$Comp
+L Device:Battery_Cell BT?
+U 1 1 5DC84BFF
+P 2200 2400
+F 0 "BT?" H 2318 2496 50  0000 L CNN
+F 1 "Battery_Cell" H 2318 2405 50  0000 L CNN
+F 2 "" V 2200 2460 50  0001 C CNN
+F 3 "~" V 2200 2460 50  0001 C CNN
+	1    2200 2400
+	1    0    0    -1
+$EndComp
+Text HLabel 2200 1700 1    50   Input ~ 0
+VDD
+Text HLabel 2200 2550 3    50   Input ~ 0
+GND
+Text HLabel 5650 2550 1    50   Input ~ 0
+VDD
+Text HLabel 5650 4650 3    50   Input ~ 0
+GND
+$Comp
+L Device:C C?
+U 1 1 5DC86BF6
+P 4950 4500
+F 0 "C?" H 5065 4546 50  0000 L CNN
+F 1 "0.1 uF" H 5065 4455 50  0000 L CNN
+F 2 "" H 4988 4350 50  0001 C CNN
+F 3 "~" H 4950 4500 50  0001 C CNN
+	1    4950 4500
+	1    0    0    -1
+$EndComp
+Text HLabel 4950 4700 3    50   Input ~ 0
+GND
+Wire Wire Line
+	8450 2250 8400 2250
+Wire Wire Line
+	8400 2150 8450 2150
+Wire Wire Line
+	8450 2150 8450 2250
+Wire Wire Line
+	8500 2150 8450 2150
+Connection ~ 8450 2150
+Text HLabel 8500 2150 2    50   Input ~ 0
+VDD
+Text HLabel 8450 2350 2    50   Input ~ 0
+GND
+Text HLabel 7550 2450 0    50   Input ~ 0
+GND
+Text HLabel 7550 2250 0    50   Input ~ 0
+SDA
+Text HLabel 7550 1950 0    50   Input ~ 0
+SCL
+$Comp
+L Device:R R?
+U 1 1 5DC886AF
+P 3650 4200
+F 0 "R?" V 3450 4200 50  0000 C CNN
+F 1 "10 K" V 3534 4200 50  0000 C CNN
+F 2 "" V 3580 4200 50  0001 C CNN
+F 3 "~" H 3650 4200 50  0001 C CNN
+	1    3650 4200
+	0    1    1    0
+$EndComp
+Text HLabel 3450 4200 0    50   Input ~ 0
+VDD
+$Comp
+L Switch:SW_SPST SW?
+U 1 1 5DC8A329
+P 2200 1950
+F 0 "SW?" V 2154 2048 50  0000 L CNN
+F 1 "SW_SPST" V 2245 2048 50  0000 L CNN
+F 2 "" H 2200 1950 50  0001 C CNN
+F 3 "~" H 2200 1950 50  0001 C CNN
+	1    2200 1950
+	0    1    1    0
+$EndComp
+Text HLabel 3850 4200 2    50   Input ~ 0
+NRESET
+Text HLabel 5000 4200 0    50   Input ~ 0
+NRESET
+$Comp
+L Connector_Generic:Conn_01x04 J?
+U 1 1 5DC8CC4A
+P 2250 3750
+F 0 "J?" H 2168 4067 50  0000 C CNN
+F 1 "Conn_01x04" H 2168 3976 50  0000 C CNN
+F 2 "" H 2250 3750 50  0001 C CNN
+F 3 "~" H 2250 3750 50  0001 C CNN
+	1    2250 3750
+	-1   0    0    -1
+$EndComp
+Text HLabel 2500 3650 2    50   Input ~ 0
+VDD
+Text HLabel 2500 3750 2    50   Input ~ 0
+SWIM
+Text HLabel 6300 3300 2    50   Input ~ 0
+SWIM
+Text HLabel 2500 3850 2    50   Input ~ 0
+NRESET
+Text HLabel 2500 3950 2    50   Input ~ 0
+GND
+$Comp
+L Device:C C?
+U 1 1 5DC8FA3A
+P 8950 2400
+F 0 "C?" H 9065 2446 50  0000 L CNN
+F 1 "0.1 uF" H 9065 2355 50  0000 L CNN
+F 2 "" H 8988 2250 50  0001 C CNN
+F 3 "~" H 8950 2400 50  0001 C CNN
+	1    8950 2400
+	1    0    0    -1
+$EndComp
+Text HLabel 8950 2200 1    50   Input ~ 0
+VDD
+Text HLabel 8950 2600 3    50   Input ~ 0
+GND
+$Comp
+L Device:C C?
+U 1 1 5DC90E07
+P 6100 2100
+F 0 "C?" H 6215 2146 50  0000 L CNN
+F 1 "C" H 6215 2055 50  0000 L CNN
+F 2 "" H 6138 1950 50  0001 C CNN
+F 3 "~" H 6100 2100 50  0001 C CNN
+	1    6100 2100
+	1    0    0    -1
+$EndComp
+Text HLabel 6100 2300 3    50   Input ~ 0
+GND
+Wire Wire Line
+	6100 1950 6100 1900
+Text HLabel 6100 1900 1    50   Input ~ 0
+VDD
+Wire Wire Line
+	6100 2300 6100 2250
+Wire Wire Line
+	5650 2550 5650 2600
+Wire Wire Line
+	5000 3300 5050 3300
+Wire Wire Line
+	5050 3400 5000 3400
+Wire Wire Line
+	6300 3300 6250 3300
+Wire Wire Line
+	5650 4650 5650 4600
+Wire Wire Line
+	5000 4200 5050 4200
+Wire Wire Line
+	4950 4350 4950 4300
+Wire Wire Line
+	4950 4300 5050 4300
+Wire Wire Line
+	4950 4700 4950 4650
+Wire Wire Line
+	3850 4200 3800 4200
+Wire Wire Line
+	3450 4200 3500 4200
+Wire Wire Line
+	2200 2550 2200 2500
+Wire Wire Line
+	2200 2150 2200 2200
+Wire Wire Line
+	2200 1700 2200 1750
+Wire Wire Line
+	2450 3650 2500 3650
+Wire Wire Line
+	2500 3750 2450 3750
+Wire Wire Line
+	2450 3850 2500 3850
+Wire Wire Line
+	2500 3950 2450 3950
+Wire Wire Line
+	7550 1950 7600 1950
+Wire Wire Line
+	7550 2250 7600 2250
+Wire Wire Line
+	7600 2450 7550 2450
+Wire Wire Line
+	8450 2350 8400 2350
+Wire Wire Line
+	8950 2600 8950 2550
+Wire Wire Line
+	8950 2250 8950 2200
 $EndSCHEMATC

Commit message: start adding led matrix
Parts:
- added D? (x16): LED, symbol Device:LED
- added R? (x4): 600, symbol Device:R
- added R? (x12): R, symbol Device:R
- C?: value C -> 0.1 uF
Connections:
- net ROW0: now reaches U?.10 (PC3)
- net ROW0: now also D?.1 (K)
- net ROW1: now reaches U?.11 (PC4)
- net ROW2: now reaches U?.12 (PC5)
- net ROW3: now reaches U?.13 (PC6)
- net COL0: now reaches U?.16 (PD2)
- net COL1: now reaches U?.17 (PD3)
- net COL2: now reaches U?.18 (PD4)
- net COL2: now also R?.1
- net COL3: now reaches U?.19 (PD5)
- net COL3: now also R?.1, R?.1, R?.1, R?.1
- new net: D?.2 (A), R?.2 (x16)
